Commit message: SITL: real-scale world (patched with PX4 sensor systems), front RGBD camera, window_detect
Co-Authored-By: Claude Opus 5 <noreply@anthropic.com>

File: sim/sim_drone.urdf.xacro (robot description, xacro)
@@ -25,3 +25,26 @@
     </sensor>
   </gazebo>
+  <!-- Front RealSense D435i stand-in: colour + depth from one rgbd_camera, so
+       depth is pixel-aligned to colour exactly like aligned_depth_to_color.
+       Mounted where the launch files put the real one (cam_x 0.105, cam_z -0.04). -->
+  <joint name="front_cam_joint" type="fixed">
+    <parent link="base_link"/>
+    <child link="front_cam_link"/>
+    <origin xyz="0.105 0 -0.04" rpy="0 0 0"/>
+  </joint>
+  <link name="front_cam_link">
+    <inertial><mass value="0.01"/>
+      <inertia ixx="1e-6" ixy="0" ixz="0" iyy="1e-6" iyz="0" izz="1e-6"/></inertial>
+  </link>
+  <gazebo reference="front_cam_link">
+    <sensor name="front_cam" type="rgbd_camera">
+      <topic>front_cam</topic>
+      <update_rate>15</update_rate>
+      <camera>
+        <horizontal_fov>1.204</horizontal_fov>
+        <image><width>640</width><height>480</height><format>R8G8B8</format></image>
+        <clip><near>0.1</near><far>10</far></clip>
+      </camera>
+    </sensor>
+  </gazebo>
 </robot>

Commit message: SITL: LDS-01 2D lidar + lidar_loc pipeline (/lidar/odom_kf), dimmed lighting
Co-Authored-By: Claude Opus 5 <noreply@anthropic.com>

File: sim/sim_drone.urdf.xacro (robot description, xacro)
@@ -48,3 +48,29 @@
     </sensor>
   </gazebo>
+  <!-- TurtleBot LDS-01 2D lidar: 360 deg, 1 deg steps, 0.12-3.5 m, ~5 Hz,
+       mounted 0.135 m above the body so the scan plane sits at flight height
+       + 0.135 (lidar_arena.yaml's mount_xyz). Read by lidar_loc's
+       gz_lidar_node on its default gz topic. -->
+  <joint name="lidar_2d_joint" type="fixed">
+    <parent link="base_link"/>
+    <child link="lidar_2d_link"/>
+    <origin xyz="0 0 0.135" rpy="0 0 0"/>
+  </joint>
+  <link name="lidar_2d_link">
+    <inertial><mass value="0.01"/>
+      <inertia ixx="1e-6" ixy="0" ixz="0" iyy="1e-6" iyz="0" izz="1e-6"/></inertial>
+  </link>
+  <gazebo reference="lidar_2d_link">
+    <sensor name="lidar_2d" type="gpu_lidar">
+      <topic>lidar_2d_v2/scan</topic>
+      <update_rate>5.5</update_rate>
+      <lidar>
+        <scan><horizontal><samples>360</samples><resolution>1</resolution>
+          <min_angle>-3.14159</min_angle><max_angle>3.14159</max_angle></horizontal></scan>
+        <range><min>0.12</min><max>3.5</max><resolution>0.015</resolution></range>
+        <noise><type>gaussian</type><mean>0</mean><stddev>0.01</stddev></noise>
+      </lidar>
+      <always_on>1</always_on>
+    </sensor>
+  </gazebo>
 </robot>
